File: KiCAD/LED driver switch/_autosave-LED driver switch.kicad_sch (KiCad schematic)
At the start: 37 parts, among them J1 3x Banana Jack, J2 USB Jack, J3 Conn_01x04_Pin, J4 TTl-RS232, J5 JST-XH Connector, J6 8P8C_Shielded, Q1 TN2124, Q2 PMOS, SW1 Door interlock, SW2 Door interlock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

Commit message: Current setup
Parts:
- removed SW2, SW3: Door interlock, symbol Switch:SW_Reed
Connections:
- net Enclosure safety interlock1: no longer names the net of U8.29 (12_A11)
- net Enclosure safety interlock2: no longer names the net of U8.28 (~11)
Changed lines of the file:
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@@
-    (effects (font (size 1.27 1.27)) (justify left bottom))
-  )
-  (label "Enclosure safety interlock1" (at 92.71 146.05 0) (fields_autoplaced)
     (effects (font (size 1.27 1.27)) (justify left bottom))
   )
@@
     (effects (font (size 1.27 1.27)) (justify right bottom))
   )
-  (label "Enclosure safety interlock1" (at 254 45.72 0) (fields_autoplaced)
-    (effects (font (size 1.27 1.27)) (justify left bottom))
-  )
   (label "Power supply+" (at 182.88 59.69 0) (fields_autoplaced)
     (effects (font (size 1.27 1.27)) (justify left bottom))
@@
   )
   (label "LED+" (at 97.79 96.52 0) (fields_autoplaced)
-    (effects (font (size 1.27 1.27)) (justify left bottom))
-  )
-  (label "Enclosure safety interlock2" (at 254 48.26 0) (fields_autoplaced)
     (effects (font (size 1.27 1.27)) (justify left bottom))
   )
@@
   )
   (label "RS-232 Tx" (at 254 53.34 0) (fields_autoplaced)
-    (effects (font (size 1.27 1.27)) (justify left bottom))
-  )
-  (label "Enclosure safety interlock2" (at 92.71 153.67 0) (fields_autoplaced)
     (effects (font (size 1.27 1.27)) (justify left bottom))
   )
@@
     )
   )
-  (symbol (lib_id "power:GND") (at 82.55 146.05 270) (unit 1)
-    (in_bom yes) (on_board yes) (dnp no) (fields_autoplaced)
-    (property "Reference" "#PWR028" (at 76.2 146.05 0)
-      (effects (font (size 1.27 1.27)) hide)
-    )
-    (property "Value" "GND" (at 79.3751 146.3668 90)
-      (effects (font (size 1.27 1.27)) (justify right))
-    )
-    (property "Footprint" "" (at 82.55 146.05 0)
-      (effects (font (size 1.27 1.27)) hide)
-    )
-    (property "Datasheet" "" (at 82.55 146.05 0)
-      (effects (font (size 1.27 1.27)) hide)
-    )
-    (pin "1")
-    (instances
-      (project "LED driver switch"
-        (path "/81d2b430-cb23-414b-8bc0-910fdb221d10"
-          (reference "#PWR028") (unit 1)
-        )
-      )
-      (project "Dual encoder controller"
-        (path "/f63253f1-d78d-4fac-a266-90df8fae5286"
-          (reference "#PWR09") (unit 1)
-        )
-      )
-    )
-  )
   (symbol (lib_id "Custom:Vref") (at 203.2 38.1 0) (mirror y) (unit 1)
     (in_bom yes) (on_board yes) (dnp no)
@@
         (path "/f63253f1-d78d-4fac-a266-90df8fae5286"
           (reference "#PWR010") (unit 1)
-        )
-      )
-    )
-  )
-  (symbol (lib_id "power:GND") (at 82.55 153.67 270) (unit 1)
-    (in_bom yes) (on_board yes) (dnp no) (fields_autoplaced)
-    (property "Reference" "#PWR029" (at 76.2 153.67 0)
-      (effects (font (size 1.27 1.27)) hide)
-    )
-    (property "Value" "GND" (at 79.3751 153.9868 90)
-      (effects (font (size 1.27 1.27)) (justify right))
-    )
-    (property "Footprint" "" (at 82.55 153.67 0)
-      (effects (font (size 1.27 1.27)) hide)
-    )
-    (property "Datasheet" "" (at 82.55 153.67 0)
-      (effects (font (size 1.27 1.27)) hide)
-    )
-    (pin "1")
-    (instances
-      (project "LED driver switch"
-        (path "/81d2b430-cb23-414b-8bc0-910fdb221d10"
-          (reference "#PWR029") (unit 1)
-        )
-      )
-      (project "Dual encoder controller"
-        (path "/f63253f1-d78d-4fac-a266-90df8fae5286"
-          (reference "#PWR09") (unit 1)
         )
       )
@@
     )
   )
-  (symbol (lib_id "Switch:SW_Reed") (at 87.63 153.67 0) (unit 1)
-    (in_bom yes) (on_board yes) (dnp no) (fields_autoplaced)
-    (property "Reference" "SW3" (at 87.63 149.2631 0)
-      (effects (font (size 1.27 1.27)))
-    )
-    (property "Value" "Door interlock" (at 87.63 151.1841 0)
-      (effects (font (size 1.27 1.27)))
-    )
-    (property "Footprint" "" (at 87.63 153.67 0)
-      (effects (font (size 1.27 1.27)) hide)
-    )
-    (property "Datasheet" "https://comus-intl.com/wp-content/uploads/2019/03/RI-02SMDM.pdf" (at 87.63 153.67 0)
-      (effects (font (size 1.27 1.27)) hide)
-    )
-    (property "Manufacturer" "Comus International" (at 87.63 153.67 0)
-      (effects (font (size 1.27 1.27)) hide)
-    )
-    (property "Part" "RI-02SMDM-1520-G1" (at 87.63 153.67 0)
-      (effects (font (size 1.27 1.27)) hide)
-    )
-    (pin "1")
-    (pin "2")
-    (instances
-      (project "LED driver switch"
-        (path "/81d2b430-cb23-414b-8bc0-910fdb221d10"
-          (reference "SW3") (unit 1)
-        )
-      )
-    )
-  )
   (symbol (lib_id "power:+5V") (at 231.14 38.1 90) (unit 1)
     (in_bom yes) (on_board yes) (dnp no)
@@
         )
       )
-    )
-  )
-  (symbol (lib_id "Switch:SW_Reed") (at 87.63 146.05 0) (unit 1)
-    (in_bom yes) (on_board yes) (dnp no) (fields_autoplaced)
-    (property "Reference" "SW2" (at 87.63 141.6431 0)
-      (effects (font (size 1.27 1.27)))
-    )
-    (property "Value" "Door interlock" (at 87.63 143.5641 0)
-      (effects (font (size 1.27 1.27)))
-    )
-    (property "Footprint" "" (at 87.63 146.05 0)
-      (effects (font (size 1.27 1.27)) hide)
-    )
-    (property "Datasheet" "https://comus-intl.com/wp-content/uploads/2019/03/RI-02SMDM.pdf" (at 87.63 146.05 0)
-      (effects (font (size 1.27 1.27)) hide)
-    )
-    (property "Manufacturer" "Comus International" (at 87.63 146.05 0)
-      (effects (font (size 1.27 1.27)) hide)
-    )
-    (property "Part" "RI-02SMDM-1520-G1" (at 87.63 146.05 0)
-      (effects (font (size 1.27 1.27)) hide)
-    )
-    (pin "1")
-    (pin "2")
-    (instances
-      (project "LED driver switch"
-        (path "/81d2b430-cb23-414b-8bc0-910fdb221d10"
-          (reference "SW2") (unit 1)
-        )
-      )
