File: KiCAD/LED driver switch/LED driver switch.kicad_sch (KiCad schematic)
At the start: 46 parts, among them J1 USB Jack, J2 3x Banana Jack, J3 Conn_Coaxial, J4 8P8C_Shielded, J5 Conn_01x04_Pin, J6 TTl-RS232, J7 Wires to LED, J8 JST-XH Connector, Q1 PMOS, Q2 TN2124, SW1 SW_Push_LED, SW2 Door interlock, SW3 Door interlock, U2 4.096V

Commit message: Move cap and standoff, fix cap polarity, add jumper 0V to GND
Parts:
- added JP1: Jumper_2_Open, Jumper:SolderJumper-2_P1.3mm_Open_Pad1.0x1.5mm, symbol Jumper:Jumper_2_Open
- added SYM3: Logo_Open_Hardware_Small, Symbol:OSHW-Logo2_7.3x6mm_SilkScreen, symbol Graphic:Logo_Open_Hardware_Small
Connections:
- net 0-200V: now also C4.1, C4.2; no longer C4.3, C4.4
- net Earth_Protective: now also JP1.1 (A)
- net GND: now also C4.3, C4.4, JP1.2 (B); no longer C4.1, C4.2
Other:
- moved on the sheet: C4
Changed lines of the file:
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@@
   (junction (at 119.38 62.23) (diameter 0) (color 0 0 0 0)
   )
+  (junction (at 92.71 77.47) (diameter 0) (color 0 0 0 0)
+  )
   (junction (at 166.37 50.8) (diameter 0) (color 0 0 0 0)
   )
   (junction (at 147.32 43.18) (diameter 0) (color 0 0 0 0)
   )
-  (junction (at 96.52 77.47) (diameter 0) (color 0 0 0 0)
-  )
   (junction (at 132.08 62.23) (diameter 0) (color 0 0 0 0)
   )
@@
   (junction (at 127 62.23) (diameter 0) (color 0 0 0 0)
   )
+  (junction (at 95.25 77.47) (diameter 0) (color 0 0 0 0)
+  )
   (junction (at 233.68 40.64) (diameter 0) (color 0 0 0 0)
   )
@@
   (junction (at 173.99 48.26) (diameter 0) (color 0 0 0 0)
   )
-  (junction (at 99.06 62.23) (diameter 0) (color 0 0 0 0)
-  )
   (junction (at 95.25 90.17) (diameter 0) (color 0 0 0 0)
   )
@@
   (junction (at 87.63 77.47) (diameter 0) (color 0 0 0 0)
   )
+  (junction (at 95.25 62.23) (diameter 0) (color 0 0 0 0)
+  )
   (junction (at 74.93 62.23) (diameter 0) (color 0 0 0 0)
   )
@@
   (junction (at 59.69 36.83) (diameter 0) (color 0 0 0 0)
   )
+  (junction (at 92.71 62.23) (diameter 0) (color 0 0 0 0)
+  )
   (junction (at 243.84 38.1) (diameter 0) (color 0 0 0 0)
   )
   (junction (at 243.84 40.64) (diameter 0) (color 0 0 0 0)
-  )
-  (junction (at 99.06 77.47) (diameter 0) (color 0 0 0 0)
-  )
-  (junction (at 96.52 62.23) (diameter 0) (color 0 0 0 0)
   )
   (junction (at 166.37 99.06) (diameter 0) (color 0 0 0 0)
@@
     (stroke (width 0) (type default))
   )
-  (wire (pts (xy 96.52 77.47) (xy 99.06 77.47))
-    (stroke (width 0) (type default))
-  )
   (wire (pts (xy 166.37 106.68) (xy 170.18 106.68))
     (stroke (width 0) (type default))
@@
     (stroke (width 0) (type default))
   )
+  (wire (pts (xy 92.71 62.23) (xy 95.25 62.23))
+    (stroke (width 0) (type default))
+  )
   (wire (pts (xy 229.87 48.26) (xy 229.87 38.1))
     (stroke (width 0) (type default))
   )
-  (wire (pts (xy 87.63 77.47) (xy 96.52 77.47))
-    (stroke (width 0) (type default))
-  )
   (wire (pts (xy 245.11 38.1) (xy 245.11 41.91))
     (stroke (width 0) (type default))
@@
     (stroke (width 0) (type default))
   )
-  (wire (pts (xy 74.93 62.23) (xy 96.52 62.23))
-    (stroke (width 0) (type default))
-  )
   (wire (pts (xy 229.87 38.1) (xy 233.68 38.1))
     (stroke (width 0) (type default))
@@
     (stroke (width 0) (type default))
   )
+  (wire (pts (xy 95.25 77.47) (xy 105.41 77.47))
+    (stroke (width 0) (type default))
+  )
   (wire (pts (xy 233.68 40.64) (xy 233.68 43.18))
     (stroke (width 0) (type default))
@@
     (stroke (width 0) (type default))
   )
-  (wire (pts (xy 96.52 62.23) (xy 99.06 62.23))
-    (stroke (width 0) (type default))
-  )
   (wire (pts (xy 173.99 50.8) (xy 173.99 48.26))
     (stroke (width 0) (type default))
@@
     (stroke (width 0) (type default))
   )
+  (wire (pts (xy 95.25 62.23) (xy 109.22 62.23))
+    (stroke (width 0) (type default))
+  )
   (wire (pts (xy 259.715 41.91) (xy 259.715 46.355))
     (stroke (width 0) (type default))
   )
+  (wire (pts (xy 92.71 77.47) (xy 95.25 77.47))
+    (stroke (width 0) (type default))
+  )
   (wire (pts (xy 109.22 62.23) (xy 109.22 67.31))
     (stroke (width 0) (type default))
@@
     (stroke (width 0) (type default))
   )
-  (wire (pts (xy 99.06 62.23) (xy 109.22 62.23))
+  (wire (pts (xy 74.93 62.23) (xy 92.71 62.23))
+    (stroke (width 0) (type default))
+  )
+  (wire (pts (xy 125.73 44.45) (xy 125.73 45.72))
     (stroke (width 0) (type default))
   )
@@
     (stroke (width 0) (type default))
   )
-  (wire (pts (xy 99.06 77.47) (xy 105.41 77.47))
+  (wire (pts (xy 87.63 77.47) (xy 92.71 77.47))
     (stroke (width 0) (type default))
   )
@@
         (path "/81d2b430-cb23-414b-8bc0-910fdb221d10"
           (reference "C1") (unit 1)
+        )
+      )
+    )
+  )
+  (symbol (lib_id "power:GND") (at 125.73 45.72 0) (unit 1)
+    (in_bom yes) (on_board yes) (dnp no)
+    (property "Reference" "#PWR029" (at 125.73 52.07 0)
+      (effects (font (size 1.27 1.27)) hide)
+    )
+    (property "Value" "GND" (at 125.73 49.53 0)
+      (effects (font (size 1.27 1.27)))
+    )
+    (property "Footprint" "" (at 125.73 45.72 0)
+      (effects (font (size 1.27 1.27)) hide)
+    )
+    (property "Datasheet" "" (at 125.73 45.72 0)
+      (effects (font (size 1.27 1.27)) hide)
+    )
+    (pin "1")
+    (instances
+      (project "LED driver switch"
+        (path "/81d2b430-cb23-414b-8bc0-910fdb221d10"
+          (reference "#PWR029") (unit 1)
+        )
+      )
+      (project "Dual encoder controller"
+        (path "/f63253f1-d78d-4fac-a266-90df8fae5286"
+          (reference "#PWR?") (unit 1)
         )
       )
@@
     )
   )
+  (symbol (lib_id "Graphic:Logo_Open_Hardware_Small") (at 96.52 46.99 0) (unit 1)
+    (in_bom no) (on_board yes) (dnp no) (fields_autoplaced)
+    (property "Reference" "SYM3" (at 96.52 40.005 0)
+      (effects (font (size 1.27 1.27)) hide)
+    )
+    (property "Value" "Logo_Open_Hardware_Small" (at 96.52 52.705 0)
+      (effects (font (size 1.27 1.27)) hide)
+    )
+    (property "Footprint" "Symbol:OSHW-Logo2_7.3x6mm_SilkScreen" (at 96.52 46.99 0)
+      (effects (font (size 1.27 1.27)) hide)
+    )
+    (property "Datasheet" "~" (at 96.52 46.99 0)
+      (effects (font (size 1.27 1.27)) hide)
+    )
+    (property "Sim.Enable" "0" (at 96.52 46.99 0)
+      (effects (font (size 1.27 1.27)) hide)
+    )
+    (property "Manufacturer" "" (at 96.52 46.99 0)
+      (effects (font (size 1.27 1.27)) hide)
+    )
+    (property "Part" "" (at 96.52 46.99 0)
+      (effects (font (size 1.27 1.27)) hide)
+    )
+    (instances
+      (project "LED driver switch"
+        (path "/81d2b430-cb23-414b-8bc0-910fdb221d10"
+          (reference "SYM3") (unit 1)
+        )
+      )
+    )
+  )
+  (symbol (lib_id "power:Earth_Protective") (at 115.57 44.45 0) (unit 1)
+    (in_bom yes) (on_board yes) (dnp no) (fields_autoplaced)
+    (property "Reference" "#PWR028" (at 121.92 50.8 0)
+      (effects (font (size 1.27 1.27)) hide)
+    )
+    (property "Value" "Earth_Protective" (at 127 48.26 0)
+      (effects (font (size 1.27 1.27)) hide)
+    )
+    (property "Footprint" "" (at 115.57 46.99 0)
+      (effects (font (size 1.27 1.27)) hide)
+    )
+    (property "Datasheet" "~" (at 115.57 46.99 0)
+      (effects (font (size 1.27 1.27)) hide)
+    )
+    (pin "1")
+    (instances
+      (project "LED driver switch"
+        (path "/81d2b430-cb23-414b-8bc0-910fdb221d10"
+          (reference "#PWR028") (unit 1)
+        )
+      )
+    )
+  )
   (symbol (lib_id "power:GND") (at 195.58 45.72 270) (unit 1)
     (in_bom yes) (on_board yes) (dnp no) (fields_autoplaced)
@@
     )
   )
-  (symbol (lib_id "Custom:ALF20G223EH063") (at 96.52 82.55 90) (unit 1)
-    (in_bom yes) (on_board yes) (dnp no) (fields_autoplaced)
-    (property "Reference" "C4" (at 93.2815 69.103 90)
+  (symbol (lib_id "Custom:ALF20G223EH063") (at 95.25 57.15 270) (unit 1)
+    (in_bom yes) (on_board yes) (dnp no) (fields_autoplaced)
+    (property "Reference" "C4" (at 98.4885 69.103 90)
       (effects (font (size 1.524 1.524)) (justify left))
     )
-    (property "Value" "3mF" (at 93.2815 71.3572 90)
+    (property "Value" "3mF" (at 98.4885 71.3572 90)
       (effects (font (size 1.524 1.524)) (justify left))
     )
-    (property "Footprint" "Custom footprints:ALF20G302KP400" (at 108.585 68.58 0)
+    (property "Footprint" "Custom footprints:ALF20G302KP400" (at 83.185 71.12 0)
       (effects (font (size 1.27 1.27) italic) hide)
     )
-    (property "Datasheet" "ALF20G223EH063" (at 104.775 70.485 0)
+    (property "Datasheet" "https://mm.digikey.com/Volume0/opasdata/d220001/medias/docus/43/ALF20_ALF40_10-17-17.pdf" (at 86.995 69.215 0)
       (effects (font (size 1.27 1.27) italic) hide)
     )
-    (property "Manufacturer" "KEMET" (at 96.52 82.55 0)
-      (effects (font (size 1.27 1.27)) hide)
-    )
-    (property "Part" "ALF20G302KP400" (at 96.52 82.55 0)
+    (property "Manufacturer" "KEMET" (at 95.25 57.15 0)
+      (effects (font (size 1.27 1.27)) hide)
+    )
+    (property "Part" "ALF20G302KP400" (at 95.25 57.15 0)
       (effects (font (size 1.27 1.27)) hide)
     )
@@
         )
       )
+    )
+  )
+  (symbol (lib_id "Jumper:Jumper_2_Open") (at 120.65 44.45 0) (unit 1)
+    (in_bom yes) (on_board yes) (dnp no) (fields_autoplaced)
+    (property "Reference" "JP1" (at 120.65 39.7891 0)
+      (effects (font (size 1.27 1.27)))
+    )
+    (property "Value" "Jumper_2_Open" (at 120.65 41.7101 0)
+      (effects (font (size 1.27 1.27)))
+    )
+    (property "Footprint" "Jumper:SolderJumper-2_P1.3mm_Open_Pad1.0x1.5mm" (at 120.65 44.45 0)
+      (effects (font (size 1.27 1.27)) hide)
+    )
+    (property "Datasheet" "~" (at 120.65 44.45 0)
+      (effects (font (size 1.27 1.27)) hide)
+    )
+    (property "Manufacturer" "" (at 120.65 44.45 0)
+      (effects (font (size 1.27 1.27)) hide)
+    )
+    (property "Part" "" (at 120.65 44.45 0)
+      (effects (font (size 1.27 1.27)) hide)
+    )
+    (pin "1")
+    (pin "2")
+    (instances
+      (project "LED driver switch"
+        (path "/81d2b430-cb23-414b-8bc0-910fdb221d10"
+          (reference "JP1") (unit 1)
+        )
+      )

Commit message: Move high voltage away from board edge - build enclosure model
Changed lines of the file:
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@@
   (no_connect (at 209.55 82.55))
   (no_connect (at 195.58 58.42))
-  (no_connect (at 304.165 6.35))
+  (no_connect (at 276.86 20.32))
   (no_connect (at 218.44 55.88))
   (no_connect (at 195.58 38.1))
@@
   (no_connect (at 243.84 35.56))
   (no_connect (at 218.44 60.96))
-  (no_connect (at 304.165 13.97))
+  (no_connect (at 276.86 27.94))
   (no_connect (at 195.58 63.5))
   (no_connect (at 195.58 66.04))
   (no_connect (at 195.58 50.8))
-  (no_connect (at 296.545 21.59))
+  (no_connect (at 269.24 35.56))
   (no_connect (at 218.44 68.58))
   (no_connect (at 218.44 45.72))
@@
   (no_connect (at 218.44 43.18))
   (no_connect (at 218.44 66.04))
-  (no_connect (at 294.005 21.59))
+  (no_connect (at 266.7 35.56))
   (no_connect (at 195.58 68.58))
-  (no_connect (at 304.165 11.43))
+  (no_connect (at 276.86 25.4))
   (no_connect (at 233.68 35.56))
   (wire (pts (xy 95.25 85.09) (xy 105.41 85.09))

Commit message: Add high voltage slots
Parts:
- removed H1, H3: Standoff, Custom footprints:8-32 Standoff, symbol Mechanical:MountingHole_Pad
- removed JP1: Jumper_2_Open, Jumper:SolderJumper-2_P1.3mm_Open_Pad1.0x1.5mm, symbol Jumper:Jumper_2_Open
- removed SW2: Door interlock, symbol Switch:SW_Reed
- added C6: 1nF, Capacitor_SMD:C_0603_1608Metric, symbol Device:C_Small
- added H1, H3: Standoff, Custom footprints:8-32 Isolated Hole, symbol Mechanical:MountingHole
- added LS1: Speaker_Crystal, Custom footprints:XDCR_SMT-0940-T-3V-R, symbol Device:Speaker_Crystal
- added MK1: Microphone, symbol Device:Microphone_Condenser
- J2: footprint Connector_Wire:SolderWire-0.15sqmm_1x03_P4mm_D0.5mm_OD1.5mm -> Custom footprints:SolderWire-0.5sqmm_1x03_P4.6mm_D0.9mm_OD2.1mm - HV Slot
- J4: footprint Custom footprints:BEL_SS71800-019F -> Custom footprints:BEL_SS71800-019F - HV Slot
- LA1: footprint Connector_Wire:SolderWire-0.1sqmm_1x02_P3.6mm_D0.4mm_OD1mm -> Custom footprints:SolderWire-0.5sqmm_1x02_P4.6mm_D0.9mm_OD2.1mm - HV Slot
- Q2: footprint Package_TO_SOT_SMD:SOT-23-3 -> Custom footprints:SOT-23-3 - HV Slot
- R1: footprint Resistor_SMD:R_1206_3216Metric -> Custom footprints:R_1206_3216 - HV slot
Connections:
- net Earth_Protective is gone; now on net GND: H2.1, J2.2 (Pin_2), J4.SH, N1.1 (PAD)
- net +5V: now also J4.3, MK1.1 (-)
- net Door safety interlock: now also U?.7 (20_A2); no longer U?.8 (21_A3)
- net GND: now also C6.2; no longer J4.4
- net at U?.24 (~5): now also LS1.2
- net at U?.26 (~9_A9): now also LS1.1
- removed net Trap door sensor: J4.3, U?.7 (20_A2)
- new net Audio out: C6.1, J4.4, MK1.2 (+), U?.8 (21_A3)
- no-connect marks 23 -> 21
Other:
- moved on the sheet: J7, J8

Commit message: Ordered version
Other:
- moved on the sheet: SW3
Changed lines of the file:
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@@
     (effects (font (size 1.27 1.27)) (justify left bottom))
   )
-  (label "Door safety interlock" (at 57.15 139.7 0) (fields_autoplaced)
+  (label "Door safety interlock" (at 57.15 125.73 0) (fields_autoplaced)
     (effects (font (size 1.27 1.27)) (justify left bottom))
   )
@@
     )
   )
-  (symbol (lib_id "Switch:SW_Reed") (at 52.07 139.7 0) (unit 1)
-    (in_bom yes) (on_board yes) (dnp no) (fields_autoplaced)
-    (property "Reference" "SW3" (at 52.07 135.2931 0)
-      (effects (font (size 1.27 1.27)))
-    )
-    (property "Value" "Door interlock" (at 52.07 137.2141 0)
-      (effects (font (size 1.27 1.27)))
-    )
-    (property "Footprint" "" (at 52.07 139.7 0)
-      (effects (font (size 1.27 1.27)) hide)
-    )
-    (property "Datasheet" "https://comus-intl.com/wp-content/uploads/2019/03/RI-02SMDM.pdf" (at 52.07 139.7 0)
-      (effects (font (size 1.27 1.27)) hide)
-    )
-    (property "Manufacturer" "Comus International" (at 52.07 139.7 0)
-      (effects (font (size 1.27 1.27)) hide)
-    )
-    (property "Part" "RI-02SMDM-1520-G1" (at 52.07 139.7 0)
+  (symbol (lib_id "Switch:SW_Reed") (at 52.07 125.73 0) (unit 1)
+    (in_bom yes) (on_board yes) (dnp no) (fields_autoplaced)
+    (property "Reference" "SW3" (at 52.07 121.3231 0)
+      (effects (font (size 1.27 1.27)))
+    )
+    (property "Value" "Door interlock" (at 52.07 123.2441 0)
+      (effects (font (size 1.27 1.27)))
+    )
+    (property "Footprint" "" (at 52.07 125.73 0)
+      (effects (font (size 1.27 1.27)) hide)
+    )
+    (property "Datasheet" "https://comus-intl.com/wp-content/uploads/2019/03/RI-02SMDM.pdf" (at 52.07 125.73 0)
+      (effects (font (size 1.27 1.27)) hide)
+    )
+    (property "Manufacturer" "Comus International" (at 52.07 125.73 0)
+      (effects (font (size 1.27 1.27)) hide)
+    )
+    (property "Part" "RI-02SMDM-1520-G1" (at 52.07 125.73 0)
       (effects (font (size 1.27 1.27)) hide)
     )
@@
     )
   )
-  (symbol (lib_id "Graphic:SYM_Flash_Small") (at 95.25 57.15 0) (unit 1)
+  (symbol (lib_id "Graphic:SYM_Flash_Small") (at 92.71 57.15 0) (unit 1)
     (in_bom no) (on_board yes) (dnp no) (fields_autoplaced)
-    (property "Reference" "SYM2" (at 92.964 57.15 90)
-      (effects (font (size 1.27 1.27)) hide)
-    )
-    (property "Value" "SYM_Flash_Small" (at 97.536 57.15 90)
-      (effects (font (size 1.27 1.27)) hide)
-    )
-    (property "Footprint" "Symbol:Symbol_Highvoltage_Type2_CopperTop_Small" (at 95.25 57.785 0)
-      (effects (font (size 1.27 1.27)) hide)
-    )
-    (property "Datasheet" "~" (at 105.41 59.69 0)
-      (effects (font (size 1.27 1.27)) hide)
-    )
-    (property "Sim.Enable" "0" (at 95.25 57.15 0)
-      (effects (font (size 1.27 1.27)) hide)
-    )
-    (property "Manufacturer" "" (at 95.25 57.15 0)
-      (effects (font (size 1.27 1.27)) hide)
-    )
-    (property "Part" "" (at 95.25 57.15 0)
+    (property "Reference" "SYM2" (at 90.424 57.15 90)
+      (effects (font (size 1.27 1.27)) hide)
+    )
+    (property "Value" "SYM_Flash_Small" (at 94.996 57.15 90)
+      (effects (font (size 1.27 1.27)) hide)
+    )
+    (property "Footprint" "Symbol:Symbol_Highvoltage_Type2_CopperTop_Small" (at 92.71 57.785 0)
+      (effects (font (size 1.27 1.27)) hide)
+    )
+    (property "Datasheet" "~" (at 102.87 59.69 0)
+      (effects (font (size 1.27 1.27)) hide)
+    )
+    (property "Sim.Enable" "0" (at 92.71 57.15 0)
+      (effects (font (size 1.27 1.27)) hide)
+    )
+    (property "Manufacturer" "" (at 92.71 57.15 0)
+      (effects (font (size 1.27 1.27)) hide)
+    )
+    (property "Part" "" (at 92.71 57.15 0)
       (effects (font (size 1.27 1.27)) hide)
     )
@@
     )
   )
-  (symbol (lib_id "Graphic:Logo_Open_Hardware_Small") (at 96.52 46.99 0) (unit 1)
+  (symbol (lib_id "Graphic:Logo_Open_Hardware_Small") (at 93.98 46.99 0) (unit 1)
     (in_bom no) (on_board yes) (dnp no) (fields_autoplaced)
-    (property "Reference" "SYM3" (at 96.52 40.005 0)
-      (effects (font (size 1.27 1.27)) hide)
-    )
-    (property "Value" "Logo_Open_Hardware_Small" (at 96.52 52.705 0)
-      (effects (font (size 1.27 1.27)) hide)
-    )
-    (property "Footprint" "Symbol:OSHW-Logo2_7.3x6mm_SilkScreen" (at 96.52 46.99 0)
-      (effects (font (size 1.27 1.27)) hide)
-    )
-    (property "Datasheet" "~" (at 96.52 46.99 0)
-      (effects (font (size 1.27 1.27)) hide)
-    )
-    (property "Sim.Enable" "0" (at 96.52 46.99 0)
-      (effects (font (size 1.27 1.27)) hide)
-    )
-    (property "Manufacturer" "" (at 96.52 46.99 0)
-      (effects (font (size 1.27 1.27)) hide)
-    )
-    (property "Part" "" (at 96.52 46.99 0)
+    (property "Reference" "SYM3" (at 93.98 40.005 0)
+      (effects (font (size 1.27 1.27)) hide)
+    )
+    (property "Value" "Logo_Open_Hardware_Small" (at 93.98 52.705 0)
+      (effects (font (size 1.27 1.27)) hide)
+    )
+    (property "Footprint" "Symbol:OSHW-Logo2_7.3x6mm_SilkScreen" (at 93.98 46.99 0)
+      (effects (font (size 1.27 1.27)) hide)
+    )
+    (property "Datasheet" "~" (at 93.98 46.99 0)
+      (effects (font (size 1.27 1.27)) hide)
+    )
+    (property "Sim.Enable" "0" (at 93.98 46.99 0)
+      (effects (font (size 1.27 1.27)) hide)
+    )
+    (property "Manufacturer" "" (at 93.98 46.99 0)
+      (effects (font (size 1.27 1.27)) hide)
+    )
+    (property "Part" "" (at 93.98 46.99 0)
       (effects (font (size 1.27 1.27)) hide)
     )
@@
     )
   )
-  (symbol (lib_id "Graphic:SYM_Flash_Small") (at 99.06 57.15 0) (unit 1)
+  (symbol (lib_id "Graphic:SYM_Flash_Small") (at 96.52 57.15 0) (unit 1)
     (in_bom no) (on_board yes) (dnp no) (fields_autoplaced)
-    (property "Reference" "SYM1" (at 96.774 57.15 90)
-      (effects (font (size 1.27 1.27)) hide)
-    )
-    (property "Value" "SYM_Flash_Small" (at 101.346 57.15 90)
-      (effects (font (size 1.27 1.27)) hide)
-    )
-    (property "Footprint" "Custom footprints:Symbol_HighVoltage" (at 99.06 57.785 0)
-      (effects (font (size 1.27 1.27)) hide)
-    )
-    (property "Datasheet" "~" (at 109.22 59.69 0)
-      (effects (font (size 1.27 1.27)) hide)
-    )
-    (property "Sim.Enable" "0" (at 99.06 57.15 0)
-      (effects (font (size 1.27 1.27)) hide)
-    )
-    (property "Manufacturer" "" (at 99.06 57.15 0)
-      (effects (font (size 1.27 1.27)) hide)
-    )
-    (property "Part" "" (at 99.06 57.15 0)
+    (property "Reference" "SYM1" (at 94.234 57.15 90)
+      (effects (font (size 1.27 1.27)) hide)
+    )
+    (property "Value" "SYM_Flash_Small" (at 98.806 57.15 90)
+      (effects (font (size 1.27 1.27)) hide)
+    )
+    (property "Footprint" "Custom footprints:Symbol_HighVoltage" (at 96.52 57.785 0)
+      (effects (font (size 1.27 1.27)) hide)
+    )
+    (property "Datasheet" "~" (at 106.68 59.69 0)
+      (effects (font (size 1.27 1.27)) hide)
+    )
+    (property "Sim.Enable" "0" (at 96.52 57.15 0)
+      (effects (font (size 1.27 1.27)) hide)
+    )
+    (property "Manufacturer" "" (at 96.52 57.15 0)
+      (effects (font (size 1.27 1.27)) hide)
+    )
+    (property "Part" "" (at 96.52 57.15 0)
       (effects (font (size 1.27 1.27)) hide)
     )
@@
     )
   )
-  (symbol (lib_id "power:GND") (at 46.99 139.7 270) (unit 1)
-    (in_bom yes) (on_board yes) (dnp no) (fields_autoplaced)
-    (property "Reference" "#PWR025" (at 40.64 139.7 0)
-      (effects (font (size 1.27 1.27)) hide)
-    )
-    (property "Value" "GND" (at 43.8151 140.0168 90)
+  (symbol (lib_id "power:GND") (at 46.99 125.73 270) (unit 1)
+    (in_bom yes) (on_board yes) (dnp no) (fields_autoplaced)
+    (property "Reference" "#PWR025" (at 40.64 125.73 0)
+      (effects (font (size 1.27 1.27)) hide)
+    )
+    (property "Value" "GND" (at 43.8151 126.0468 90)
       (effects (font (size 1.27 1.27)) (justify right))
     )
-    (property "Footprint" "" (at 46.99 139.7 0)
-      (effects (font (size 1.27 1.27)) hide)
-    )
-    (property "Datasheet" "" (at 46.99 139.7 0)
-      (effects (font (size 1.27 1.27)) hide)
-    )
+    (property "Footprint" "" (at 46.99 125.73 0)
+      (effects (font (size 1.27 1.27)) hide)
+    )
+    (property "Datasheet" "" (at 46.99 125.73 0)
+      (effects (font (size 1.27 1.27)) hide)
+    )
