File: KiCAD/LED driver switch/LED driver switch.kicad_sch (KiCad schematic)
At the start: 49 parts, among them J1 USB Jack, J2 3x Banana Jack, J3 Conn_Coaxial, J4 8P8C_Shielded, J5 Conn_01x04_Pin, J6 TTl-RS232, J7 Wires to LED, J8 JST-XH Connector, Q1 PMOS, Q2 TN2124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

Commit message: Add HV slots for mosfet
Parts:
- Q1: footprint Package_TO_SOT_SMD:TO-263-2 -> Custom footprints:TO-252-2 - HV
- R4: footprint Resistor_SMD:R_1206_3216Metric -> Custom footprints:R_1206_3216 - HV slot
Changed lines of the file:
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@@
       (effects (font (size 1.27 1.27)) (justify left))
     )
-    (property "Footprint" "Package_TO_SOT_SMD:TO-263-2" (at 116.84 73.66 0)
+    (property "Footprint" "Custom footprints:TO-252-2 - HV" (at 116.84 73.66 0)
       (effects (font (size 1.27 1.27)) hide)
     )
@@
       (effects (font (size 1.27 1.27)) (justify left))
     )
-    (property "Footprint" "Resistor_SMD:R_1206_3216Metric" (at 127.762 74.93 90)
+    (property "Footprint" "Custom footprints:R_1206_3216 - HV slot" (at 127.762 74.93 90)
       (effects (font (size 1.27 1.27)) hide)
     )
