File: KiCAD/LED driver switch/LED driver switch.kicad_sch (KiCad schematic)
At the start: 49 parts, among them J1 USB Jack, J2 3x Banana Jack, J3 Conn_Coaxial, J4 8P8C_Shielded, J5 Conn_01x04_Pin, J6 TTl-RS232, J7 Wires to LED, J8 JST-XH Connector, Q1 PMOS, Q2 TN2124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

Commit message: Update PCB to reflect current design
Parts:
- removed RN1: R_Pack08, Resistor_SMD:R_Array_Convex_8x0602, symbol Device:R_Pack08
- removed SW1: SW_Push_LED, Connector_Wire:SolderWire-0.1sqmm_1x05_P3.6mm_D0.4mm_OD1mm, symbol Custom:SW_Push_2x_LED_common_cathode
- added R10: 180, Resistor_SMD:R_0805_2012Metric, symbol Device:R
- added SW1: SW_Push_LED, Connector_Wire:SolderWire-0.5sqmm_1x04_P4.6mm_D0.9mm_OD2.1mm, symbol Custom:SW_Push_2x_LED
Connections:
- net +5V: no longer C1.1, U2.4 (SHDN), U2.6 (Vdd)
- net GND: now also SW1.2
- net Green_LED: now also SW1.4
- net Pushbutton: now also SW1.1
- net Red_LED: now also R10.1
- net reset: now reaches U?.1 (Reset)
- net reset: now also U?.25 (7)
- net Vbus: now reaches U?.31 (VBus)
- net Vbus: now also C1.1, U2.4 (SHDN), U2.6 (Vdd)
- new net: R10.2, SW1.3
- no-connect marks 21 -> 16
