File: KiCAD/Photogate Sensor/Transmissive/cyro_plunger_transmissive_photogate.kicad_sch (KiCad schematic)
At the start: 60 parts, among them J1 FFC, J2 FFC Socket, J3 USB_B_Micro, J4 UPDI socket, J5 DC Jack, J6 Conn_01x03_Socket, J7 USB_B_Micro, J8 FFC Socket, J9 Conn_01x03_Socket, Q1 Q_NMOS_GSD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

Commit message: Interrupt sync working
Connections:
- net Comp Out: now also J8.2 (Pin_2); no longer J8.7 (Pin_7)
- net D+: now also J8.8 (Pin_8); no longer J8.1 (Pin_1)
- net D-: now also J8.7 (Pin_7); no longer J8.2 (Pin_2)
- net Vusb: now also J8.1 (Pin_1); no longer J8.8 (Pin_8)
Changed lines of the file:
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@@
 	)
 	(label "Vusb"
-		(at 109.22 187.96 180)
+		(at 109.22 170.18 180)
 		(fields_autoplaced yes)
 		(effects
@@
 	)
 	(label "D+"
-		(at 109.22 170.18 180)
+		(at 109.22 187.96 180)
 		(fields_autoplaced yes)
 		(effects
@@
 	)
 	(label "D-"
-		(at 109.22 172.72 180)
+		(at 109.22 185.42 180)
 		(fields_autoplaced yes)
 		(effects
@@
 	)
 	(label "Comp Out"
-		(at 109.22 185.42 180)
+		(at 109.22 172.72 180)
 		(fields_autoplaced yes)
 		(effects
@@
 	(symbol
 		(lib_id "power:GND")
-		(at 109.22 182.88 270)
+		(at 109.22 175.26 270)
+		(mirror x)
 		(unit 1)
 		(exclude_from_sim no)
@@
 		(on_board yes)
 		(dnp no)
-		(fields_autoplaced yes)
 		(property "Reference" "#PWR047"
-			(at 102.87 182.88 0)
+			(at 102.87 175.26 0)
 			(effects
 				(font
@@
 		)
 		(property "Value" "GND"
-			(at 106.0451 182.88 90)
+			(at 106.0451 175.26 90)
 			(effects
 				(font
@@
 		)
 		(property "Footprint" ""
-			(at 109.22 182.88 0)
+			(at 109.22 175.26 0)
 			(effects
 				(font
@@
 		)
 		(property "Datasheet" ""
-			(at 109.22 182.88 0)
+			(at 109.22 175.26 0)
 			(effects
 				(font
@@
 		)
 		(property "Description" "Power symbol creates a global label with name \"GND\" , ground"
-			(at 109.22 182.88 0)
+			(at 109.22 175.26 0)
 			(effects
 				(font
@@
 	(symbol
 		(lib_id "power:GND")
-		(at 109.22 175.26 270)
+		(at 109.22 182.88 270)
+		(mirror x)
 		(unit 1)
 		(exclude_from_sim no)
@@
 		(fields_autoplaced yes)
 		(property "Reference" "#PWR041"
-			(at 102.87 175.26 0)
+			(at 102.87 182.88 0)
 			(effects
 				(font
@@
 		)
 		(property "Value" "GND"
-			(at 106.0451 175.26 90)
+			(at 106.0451 182.88 90)
 			(effects
 				(font
@@
 		)
 		(property "Footprint" ""
-			(at 109.22 175.26 0)
+			(at 109.22 182.88 0)
 			(effects
 				(font
@@
 		)
 		(property "Datasheet" ""
-			(at 109.22 175.26 0)
+			(at 109.22 182.88 0)
 			(effects
 				(font
@@
 		)
 		(property "Description" "Power symbol creates a global label with name \"GND\" , ground"
-			(at 109.22 175.26 0)
+			(at 109.22 182.88 0)
 			(effects
 				(font
@@
 	(symbol
 		(lib_id "power:+12V")
-		(at 109.22 177.8 90)
+		(at 109.22 180.34 90)
+		(mirror x)
 		(unit 1)
 		(exclude_from_sim no)
@@
 		(fields_autoplaced yes)
 		(property "Reference" "#PWR042"
-			(at 113.03 177.8 0)
+			(at 113.03 180.34 0)
 			(effects
 				(font
@@
 		)
 		(property "Value" "+12V"
-			(at 106.045 177.8 90)
+			(at 106.045 180.34 90)
 			(effects
 				(font
@@
 		)
 		(property "Footprint" ""
-			(at 109.22 177.8 0)
+			(at 109.22 180.34 0)
 			(effects
 				(font
@@
 		)
 		(property "Datasheet" ""
-			(at 109.22 177.8 0)
+			(at 109.22 180.34 0)
 			(effects
 				(font
@@
 		)
 		(property "Description" "Power symbol creates a global label with name \"+12V\""
-			(at 109.22 177.8 0)
+			(at 109.22 180.34 0)
 			(effects
 				(font
@@
 	(symbol
 		(lib_id "power:+12V")
-		(at 109.22 180.34 90)
+		(at 109.22 177.8 90)
+		(mirror x)
 		(unit 1)
 		(exclude_from_sim no)
@@
 		(fields_autoplaced yes)
 		(property "Reference" "#PWR046"
-			(at 113.03 180.34 0)
+			(at 113.03 177.8 0)
 			(effects
 				(font
@@
 		)
 		(property "Value" "+12V"
-			(at 106.045 180.34 90)
+			(at 106.045 177.8 90)
 			(effects
 				(font
@@
 		)
 		(property "Footprint" ""
-			(at 109.22 180.34 0)
+			(at 109.22 177.8 0)
 			(effects
 				(font
@@
 		)
 		(property "Datasheet" ""
-			(at 109.22 180.34 0)
+			(at 109.22 177.8 0)
 			(effects
 				(font
@@
 		)
 		(property "Description" "Power symbol creates a global label with name \"+12V\""
-			(at 109.22 180.34 0)
+			(at 109.22 177.8 0)
 			(effects
 				(font
